File: hardware/passerelle.kicad_sch (KiCad schematic)
At the start: 3 parts, among them U1 nRF5340-QKxx, U2 nRF7002-QFXX, U3 nRF9161-SIXX

Commit message: switch nRF9161 for nRF9151
Parts:
- removed U3: nRF9161-SIXX, PCM_nordic-lib-kicad-nrf9:LGA_9161_16.0x10.5mm, symbol PCM_nordic-lib-kicad-nrf9:nRF9161-SIXX
- added U3: nRF9151-LAXX, PCM_nordic-lib-kicad-nrf9:LGA_9151_12.1x11.1mm, symbol PCM_nordic-lib-kicad-nrf9:nRF9151-LAXX
Connections:
- new net: U3.1 (GND), U3.105 (GND), U3.106 (GND), U3.107 (GND), U3.108 (GND), U3.109 (GND), U3.110 (GND), U3.111 (GND), U3.112 (GND), U3.113 (GND), U3.13 (GND), U3.15 (GND), U3.20 (GND), U3.25 (GND), U3.30 (GND), U3.34 (GND), U3.36 (GND), U3.38 (GND), U3.39 (GND), U3.40 (GND), U3.41 (GND), U3.43 (GND), U3.46 (GND), U3.51 (GND), U3.55 (GND), U3.60 (GND), U3.66 (GND), U3.7 (GND), U3.71 (GND), U3.76 (GND)
Other:
- moved on the sheet: U1, U2

Commit message: ...
Connections:
- net D_P: now reaches U1.B2 (D+)
- net D_N: now reaches U1.B4 (D-)
Changed lines of the file:
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@@
 	(generator_version "10.0")
 	(paper "A2")
+	(label "D_N"
+		(at 284.48 243.84 0)
+		(effects
+			(font
+				(size 1.27 1.27)
+			)
+			(justify left bottom)
+		)
+	)
+	(label "D_P"
+		(at 284.48 246.38 0)
+		(effects
+			(font
+				(size 1.27 1.27)
+			)
+			(justify left bottom)
+		)
+	)
 	(symbol
 		(lib_id "MCU_Nordic:nRF5340-QKxx")

Commit message: power
Connections:
- net VBUS: now reaches U1.A5 (VBUS)
Other:
- added sheet power (power.kicad_sch)
Changed lines of the file:
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@@
+	)
+	(symbol
+		(lib_id "power:VDD")
+		(at 218.44 238.76 90)
+		(unit 1)
+		(body_style 1)
+		(exclude_from_sim no)
+		(in_bom yes)
+		(on_board yes)
+		(in_pos_files yes)
+		(dnp no)
+		(fields_autoplaced yes)
+		(property "Reference" "#PWR027"
+			(at 222.25 238.76 0)
+			(hide yes)
+			(show_name no)
+			(do_not_autoplace no)
+			(effects
+				(font
+					(size 1.27 1.27)
+				)
+			)
+		)
+		(property "Value" "VBUS"
+			(at 214.63 238.7599 90)
+			(show_name no)
+			(do_not_autoplace no)
+			(effects
+				(font
+					(size 1.27 1.27)
+				)
+				(justify left)
+			)
+		)
+		(property "Footprint" ""
+			(at 218.44 238.76 0)
+			(hide yes)
+			(show_name no)
+			(do_not_autoplace no)
+			(effects
+				(font
+					(size 1.27 1.27)
+				)
+			)
+		)
+		(property "Datasheet" ""
+			(at 218.44 238.76 0)
+			(hide yes)
+			(show_name no)
+			(do_not_autoplace no)
+			(effects
+				(font
+					(size 1.27 1.27)
+				)
+			)
+		)
+		(property "Description" "Power symbol creates a global label with name \"VDD\""
+			(at 218.44 238.76 0)
+			(hide yes)
+			(show_name no)
+			(do_not_autoplace no)
+			(effects
+				(font
+					(size 1.27 1.27)
+				)
+			)
+		)
+		(pin "1"
+		)
+		(instances
+			(project "passerelle"
+				(path "/e7d95599-b191-4688-bb45-304a9c2e4124"
+					(reference "#PWR027")
+					(unit 1)
+				)
+			)
+		)
 	)
 	(symbol
@@
 				)
 			)
+		)
+	)
+	(sheet
+		(at 86.36 142.748)
+		(size 53.34 70.612)
+		(exclude_from_sim no)
+		(in_bom yes)
+		(on_board yes)
+		(dnp no)
+		(fields_autoplaced yes)
+		(stroke
+			(width 0.1524)
+			(type solid)
+		)
+		(fill
+			(color 0 0 0 0)
+		)
+		(property "Sheetname" "power"
+			(at 86.36 142.0364 0)
+			(show_name no)
+			(do_not_autoplace no)
+			(effects
+				(font
+					(size 1.27 1.27)
+				)
+				(justify left bottom)
+			)
+		)
+		(property "Sheetfile" "power.kicad_sch"
+			(at 86.36 213.9446 0)
+			(show_name no)
+			(do_not_autoplace no)
+			(effects
+				(font
+					(size 1.27 1.27)
+				)
+				(justify left top)
+			)
+		)
+		(pin "VBUS" input
+			(at 139.7 148.59 0)
+			(effects
+				(font
+					(size 1.27 1.27)
+				)
+				(justify right)
+			)
+		)
+		(pin "D_N" input
+			(at 139.7 151.13 0)
+			(effects
+				(font
+					(size 1.27 1.27)
+				)
+				(justify right)
+			)
+		)
+		(pin "D_P" input
+			(at 139.7 153.67 0)
+			(effects
+				(font
+					(size 1.27 1.27)
+				)
+				(justify right)
+			)
+		)
+		(pin "SCL" input
+			(at 139.7 156.21 0)
+			(effects
+				(font
+					(size 1.27 1.27)
+				)
+				(justify right)
+			)
+		)
+		(pin "SDA" input
+			(at 139.7 158.75 0)
+			(effects
+				(font
+					(size 1.27 1.27)
+				)
+				(justify right)
+			)
+		)
+		(pin "GPIO2" input
+			(at 139.7 161.29 0)
+			(effects
+				(font
+					(size 1.27 1.27)
+				)
+				(justify right)
+			)
+		)
+		(pin "GPIO3" input
+			(at 139.7 163.83 0)
+			(effects
+				(font
+					(size 1.27 1.27)
+				)
+				(justify right)
+			)
+		)
+		(pin "GPIO4" input
+			(at 139.7 166.37 0)
+			(effects
+				(font
+					(size 1.27 1.27)
+				)
+				(justify right)
+			)
+		)
+		(pin "INT" input
+			(at 139.7 168.91 0)
+			(effects
+				(font
+					(size 1.27 1.27)
+				)
+				(justify right)
+			)
+		)
+		(pin "LSOUT" input
+			(at 139.7 171.45 0)
+			(effects
+				(font
+					(size 1.27 1.27)
+				)
+				(justify right)
+			)
+		)
+		(pin "RESET" input
+			(at 139.7 173.99 0)
+			(effects
+				(font
+					(size 1.27 1.27)
+				)
+				(justify right)
+			)
+		)
+		(pin "VBAT" input
+			(at 139.7 176.53 0)
+			(effects
+				(font
+					(size 1.27 1.27)
+				)
+				(justify right)
+			)
+		)
+		(pin "VDDIO" input
+			(at 139.7 179.07 0)
+			(effects
+				(font
+					(size 1.27 1.27)
+				)
+				(justify right)
+			)
+		)
+		(instances
+			(project "passerelle"
+				(path "/e7d95599-b191-4688-bb45-304a9c2e4124"
+					(page "2")
+				)
+			)
