File: hardware/power.kicad_sch (KiCad schematic)
At the start: 13 parts, among them J1 USB_C_Receptacle_USB2.0_16P, U4 nPM1300-QEXX

Commit message: power
Parts:
- added C15, C16, C17, C18, C19, C20: 10uF, symbol Device:C
- added D1, D3, D4: LED, symbol Device:LED
- added L1, L2: 2.2uH, symbol Device:L
- added R1: 150k, symbol Device:R
- added R2: 47k, symbol Device:R
- added SW1, SW2: SW_Push, symbol Switch:SW_Push
- added TH1: Thermistor, symbol Device:Thermistor
- renumbered C7 to C10, C4 to C11, C2 to C12, C3 to C13, C1 to C14, C6 to C8, C5 to C9, D1 to D2, J1 to J2, R1 to R3, R2 to R4, U4 to U5
Connections:
- net GND: now also J2.A1 (GND), J2.A12 (GND), J2.B1 (GND), J2.B12 (GND), C15.2, C16.2, C17.2, C18.2, C19.2, C20.2, R1.2, R2.2, SW1.1, SW2.1, TH1.2; no longer U5.16 (VSET2), U5.17 (VSET1), U5.18 (NTC), U5.28 (LSIN1/VINLDO1), U5.29 (LSOUT1/VOUTLDO1), U5.30 (LSIN2/VINLDO2), U5.31 (LSOUT2/VOUTLDO2)
- net VBUS: now reaches C10.2, C8.2, C9.2, D2.4 (VCC), J2.A4 (VBUS), J2.A9 (VBUS), J2.B4 (VBUS), J2.B9 (VBUS), U5.21 (VBUS)
- net VBUSOUT: now reaches C13.1, U5.22 (VBUSOUT)
- net GPIO3: now reaches U5.10 (GPIO3)
- net GPIO4: now reaches U5.11 (GPIO4)
- net at U5.15 (SHPHLD): now also SW1.2
- net at U5.25 (LED0): now also D4.1 (K)
- net at U5.26 (LED1): now also D1.1 (K)
- net at U5.27 (LED2): now also D3.1 (K)
- net at U5.3 (SW1): now also L2.2
- net at U5.5 (SW2): now also L1.2
- net RESET: now reaches U5.7 (GPIO0)
- net RESET: now also SW2.2
- net INT: now reaches U5.8 (GPIO1)
- net GPIO2: now reaches U5.9 (GPIO2)
- net +BATT renamed VBAT
- net VDD renamed VSYS
- net VSYS: now also U5.28 (LSIN1/VINLDO1), C16.1, C20.1, D1.2 (A), D3.2 (A), D4.2 (A); no longer U5.1 (VOUT1), U5.32 (VOUT2)
- new net: C15.1, L1.1, U5.32 (VOUT2)
- new net: C17.1, L2.1, U5.1 (VOUT1)
- new net: R1.1, U5.16 (VSET2)
- new net: R2.1, U5.17 (VSET1)
- new net: TH1.1, U5.18 (NTC)
- new net LSOUT: U5.31 (LSOUT2/VOUTLDO2)
- new net VLDO: C18.1, C19.1, U5.29 (LSOUT1/VOUTLDO1)
- new net VOUT2: U5.30 (LSIN2/VINLDO2)
- no-connect marks 13 -> 3
Other:
- moved on the sheet: C10, C11, C12, C13, C14, C8, C9, D2, R3, R4, U5
